File: ESXAR_panelize.kicad_pcb (KiCad board)
At the start: 2 copper layers, 186.7 x 61.1 mm, 66 parts, among them CON1 BARREL_JACK, J1 RJ45, J2 RJ45, P1 ANALOG, P1 CONN_01X02, P10 USB_A, P11 USB_B, P12 SERVO/INPUT, P13 ANALOG, P16 BREADBOARD_POWER, P17 SENSOR, P18 EXTIO, P19 UNIVERSAL, P2 BREADBOARD, P20 UNIVERSAL, P3 PROGRAM, P4 OPAMP EX, P5 MODEJP, P6 VCCJP, P7 GNDJP, P8 SCREW, SW1 RESET, SW2 DIN, U1 ESP-WROOM-02, U1 LM2596HV_DCDC_Module, U2 NJM4556A, U2 RASPBERRYPI_GPIO_40, U3 AUDIO_JACK, U4 MT5201-3.3N, U5 TLP222A, U6 Mini360, U7 LD1117CV33, U8 TA48M033F

Commit message: Ver.20160805 change outline, rayout, delete opamp, etc...
Parts:
- removed C4: 0.1uF, Capacitors_ThroughHole:C_Disc_D3_P2.5
- removed P4: OPAMP EX, Wire_Pads:SolderWirePad_single_0-8mmDrill
- removed R10, R11, R6, R7, R8, R9: 4.7kΩ, Discret:R1
- removed the U2 at (183.5, 129.5)
- JP1, P17, P8: moved to B.Cu
- moved J2 108.7 mm to (227.7, 57.1)
- moved U1 108.7 mm to (213.7, 83.8)
- moved CON1 108.7 mm to (158.6, 82.5)
- moved D1 108.7 mm to (227.1, 44.9)
- moved J1 108.7 mm to (227.7, 80.0)
- moved P1 108.7 mm to (219.5, 38.1)
- moved R1 108.7 mm to (215.6, 48.9)
- moved TH1 108.7 mm to (208.0, 66.0)
- moved U2 108.7 mm to (153.0, 38.9)
- moved C1 25.0 mm to (159.3, 114.0), turned to 90 degrees
- moved R1 22.3 mm to (181.5, 128.7)
- moved OSHW 22.3 mm to (141.5, 108.3)
- moved R13 16.4 mm to (181.5, 125.5)
- moved C7 11.5 mm to (168.8, 103.3), turned to 180 degrees
- moved U8 11.4 mm to (175.8, 105.6), turned to 270 degrees
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Routing:
- net Net-(C1-Pad1): track 82.6 -> 24.6 mm
- net GND: track 715.8 -> 664.1 mm, vias 10 -> 3
- net Net-(JP3-Pad1): track 117.6 -> 81.2 mm, vias 4 -> 1
- net Net-(C3-Pad1): track 30.9 -> 0.00 mm
- net Net-(P12-Pad1): track 111.1 -> 85.3 mm, vias 1 -> 3
- net +3V3: track 217.9 -> 194.9 mm, vias 6 -> 7
- net Net-(C4-Pad1): track 22.5 -> 0.00 mm
- net Net-(P13-Pad1): track 121.3 -> 101.8 mm, vias 1 -> 2
- net Net-(C1-Pad2): track 11.7 -> 31.0 mm, vias 0 -> 2
- net Net-(R10-Pad2): track 18.7 -> 0.00 mm
- net +5V: track 109.7 -> 92.3 mm, vias 3 -> 1
- net Net-(P4-Pad1): track 13.2 -> 0.00 mm
- net Net-(P18-Pad3): track 79.1 -> 69.1 mm
- net Net-(RP1-Pad5): track 43.0 -> 34.4 mm
- net Net-(P18-Pad8): track 67.4 -> 58.9 mm
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Other:
- board size 186.7 x 61.1 mm -> 93.2 x 117 mm
- board text added: "D4 5V GND"
- board text added: "ESXAR Ver.20160805"
- board text added: "L8 L7 L6 l5 L4 L3 L2 L1 D0"
- board text added: "PROGRAM▼"
- board text added: "SERVO ◀/DIN"
- board text removed: "ESXAR Ver.20160804"
- board text removed: "L8 L7 L6 L5 L4 L3 L2 L1 L0"
- board text removed: "PROGRAM"
- board text removed: "SERVO/DIN D4 5V GND"
